File: hardware/curly-memory-kicad/switches.kicad_sch (KiCad schematic)
At the start: 13 parts

Commit message: all components have part numbers
Parts:
- removed C? (x3): 100nF, Capacitor_SMD:C_0805_2012Metric_Pad1.18x1.45mm_HandSolder, symbol Device:C
- removed R? (x3): 1K, Resistor_SMD:R_0805_2012Metric_Pad1.20x1.40mm_HandSolder, symbol Device:R
- removed ROT?: RotaryEncoder_Switch, symbol Device:RotaryEncoder_Switch
- SW? (x2): value SW_MEC_5E -> FSM; footprint (none) -> Button_Switch_SMD:SW_Push_1P1T_NO_6x6mm_H9.5mm
