File: hardware/curly-memory-kicad/curly-memory-kicad.kicad_sch (KiCad schematic)
At the start: 81 parts

Commit message: output + input op amps added, simuatlion added to sim folder
Parts:
- removed C? (x14): C, symbol Device:C
- removed D? (x2): D, symbol Device:D
- removed J? (x4): AudioJack2, symbol Connector:AudioJack2
- removed J?: Conn_02x05_Odd_Even, symbol Connector_Generic:Conn_02x05_Odd_Even
- removed J? (x4): Conn_01x01_Male, symbol Connector:Conn_01x01_Male
- removed U?: L7805, symbol Regulator_Linear:L7805
- removed U?: LF33_TO220, Package_TO_SOT_THT:TO-220-3_Vertical, symbol Regulator_Linear:LF33_TO220
Connections:
- net GND: now also U?.5 (PB1); no longer U?.7 (PA1)
- net OUT_0: now also U?.7 (PA1); no longer U?.5 (PB1), U?.8 (VA)
- net OUT_1: no longer U?.6 (VB)
- net OUT_2 renamed output/OUT_2+
- net OUT_3 renamed output/OUT_3+
- new net output/OUT_0+: U?.8 (VA)
- new net output/OUT_1+: U?.6 (VB)
Other:
- sheet input_0 renamed input
- removed sheet input_1
- removed sheet input_2
- removed sheet input_3
- added sheet output (output.kicad_sch)
- added sheet power (power.kicad_sch)
- sheet input ports: added IN_0+, IN_1+, IN_2+, IN_3+; removed IN+
- note added: "Inputs connect to ADC, ADC connects to ESP32, allows audio inputs or CV inputs to be recorded 4 external input +/- 5V 4 potentiometer inputs"
- note added: "Inputs power from eurorack 10 pin Outputs various voltages for rest of circuit"
- note added: "Power"
- note removed: "Convert 12V DC to 5V DC"
- note removed: "Inputs connect to ADC, ADC connects to ESP32, allows audio inputs or CV inputs to be recorded"
- note removed: "POWER"
- moved on the sheet: C?, D?, J?, R?, RV?, U?, U?A, U?B, U?C

Commit message: schematic updated with component fields on more components
Parts:
- removed C? (x5): C, symbol Device:C
- removed R? (x7): R, symbol Device:R
- removed SW?: RotaryEncoder_Switch, symbol Device:RotaryEncoder_Switch
- removed SW? (x2): SW_MEC_5E, symbol Switch:SW_MEC_5E
- removed U?: NE5532, symbol Amplifier_Operational:NE5532
- added C?: 1uF, Capacitor_SMD:C_0805_2012Metric_Pad1.18x1.45mm_HandSolder, symbol Device:C
- added J?: Conn_01x05, Connector_PinSocket_2.54mm:PinSocket_1x05_P2.54mm_Vertical, symbol Connector_Generic:Conn_01x05
- added J?: Conn_01x01_Male, Connector_PinSocket_2.54mm:PinSocket_1x01_P2.54mm_Vertical, symbol Connector:Conn_01x01_Male
- added J?: AudioJack2, AudioJacks:Jack_3.5mm_QingPu_WQP-PJ398SM_Vertical, symbol Connector:AudioJack2_Ground_SwitchT
- added JP? (x2): Jumper_2_Open, Connector_PinHeader_2.54mm:PinHeader_1x02_P2.54mm_Vertical, symbol Jumper:Jumper_2_Open
- C? (x5): value C -> 1uF; footprint (none) -> Capacitor_SMD:C_0805_2012Metric_Pad1.18x1.45mm_HandSolder
- C? (x5): value C -> 100nF; footprint (none) -> Capacitor_SMD:C_0805_2012Metric_Pad1.18x1.45mm_HandSolder
- J?: footprint (none) -> Connector_PinSocket_2.54mm:PinSocket_1x05_P2.54mm_Vertical
- J? (x3): footprint (none) -> Connector_PinSocket_2.54mm:PinSocket_1x01_P2.54mm_Vertical
- R?: value R -> 100K; footprint (none) -> Resistor_SMD:R_0805_2012Metric_Pad1.20x1.40mm_HandSolder
- R?: value R -> 100R; footprint (none) -> Resistor_SMD:R_0805_2012Metric_Pad1.20x1.40mm_HandSolder
- R? (x4): value R -> 1K; footprint (none) -> Resistor_SMD:R_0805_2012Metric_Pad1.20x1.40mm_HandSolder
Connections:
- net GND: now also J?.T, J?.TN
- net IN_0: now also JP?.1 (A), JP?.2 (B)
- net OUT_0: now also JP?.1 (A), JP?.2 (B)
- net RES0_A1: now also R?.2
- net at U?.10 (IO25): now also J?.5 (Pin_5)
- net at U?.24 (IO2): now also J?.1 (Pin_1)
- net at U?.28 (IO17): now also J?.2 (Pin_2)
- net at U?.33 (IO21): now also J?.3 (Pin_3)
- net at U?.36 (IO22): now also J?.4 (Pin_4)
- net OUT_1 renamed RES0_W1
- net RES0_W1: now also C?.1; no longer R?.2
- new net: C?.2, J?.1 (Pin_1), J?.S, R?.2
Other:
- added sheet switches (switches.kicad_sch)
- note added: "Dry/Wet Mixer"
- note added: "Mix In_0 and Out_0 with a summing amplifier, remove jumpers and patch in any other signals"
- note added: "Switches"
- note added: "Two tactile switches and one rotary knob with switch"
- moved on the sheet: C?, D?, J?, R?, SW?, U?, U?A, U?C

Commit message: all components have part numbers
Parts:
- removed C?: 1uF, Capacitor_SMD:C_0805_2012Metric_Pad1.18x1.45mm_HandSolder, symbol Device:C
- removed U? (x2): NE5532, symbol Amplifier_Operational:NE5532
- added U?: MCP6004, Package_SO:SOIC-14_3.9x8.7mm_P1.27mm, symbol Amplifier_Operational:MCP6004
- RV? (x4): value R_POT_TRIM -> PTV09A-4225F-B203; footprint (none) -> Potentiometer_THT:Potentiometer_Bourns_PTV09A-1_Single_Vertical
- SW? (x2): value SW_MEC_5E -> FSM; footprint (none) -> Button_Switch_SMD:SW_Push_1P1T_NO_6x6mm_H9.5mm
- U?: value MCP3008 -> MCP3008-I/SL; footprint (none) -> Package_SO:SOIC-16_3.9x9.9mm_P1.27mm
- U? (x2): value MCP4822 -> MCP4822-E/SN; footprint (none) -> Package_SO:SOIC-8_3.9x4.9mm_P1.27mm
- U? (x2): value MCP42010 -> MCP42010-E/SL; footprint (none) -> Package_SO:SOIC-14_3.9x8.7mm_P1.27mm
Connections:
- net GND: now also U?.12 (+)
- net at R?.1, R?.2: now also U?.14
- net at R?.1, R?.2, R?.2: now also U?.13 (-)
- net ROT_A: no longer names the net of U?.8 (IO32)
- net ROT_B: no longer names the net of U?.12 (IO27)
- net ROT_SW: no longer names the net of U?.11 (IO26)
Other:
- sheet switches ports: added none; removed ROT_A, ROT_B, ROT_SW

Commit message: interface board added
Parts:
- J102: renamed from J?; symbol Connector_Generic:Conn_01x05 -> Connector_Generic:Conn_01x03
- gave numbers to parts that had none: 41
Connections:
- net at U102.10 (IO25): no longer J102.5 (Pin_5)
- net at U102.24 (IO2): no longer J102.1 (Pin_1)
- net at U102.28 (IO17): now also J102.1 (Pin_1); no longer J102.2 (Pin_2)
- net at U102.33 (IO21): now also J102.2 (Pin_2); no longer J102.3 (Pin_3)
- net at U102.36 (IO22): now also J102.3 (Pin_3); no longer J102.4 (Pin_4)

Commit message: all components placed on the main board
Parts:
- removed C102, C107: 1uF, Capacitor_SMD:C_0805_2012Metric_Pad1.18x1.45mm_HandSolder, symbol Device:C
- removed D101, D102, D103, D104: WS2812B, LED_SMD:LED_WS2812B_PLCC4_5.0x5.0mm_P3.2mm, symbol LED:WS2812B
- removed J103, J104, J105, J106: Conn_01x01_Male, Connector_PinSocket_2.54mm:PinSocket_1x01_P2.54mm_Vertical, symbol Connector:Conn_01x01_Male
- removed J107: AudioJack2, AudioJacks:Jack_3.5mm_QingPu_WQP-PJ398SM_Vertical, symbol Connector:AudioJack2_Ground_SwitchT
- removed JP101, JP102: Jumper_2_Open, Connector_PinHeader_2.54mm:PinHeader_1x02_P2.54mm_Vertical, symbol Jumper:Jumper_2_Open
- removed RV101, RV102, RV103, RV104: PTV09A-4225F-B203, Potentiometer_THT:Potentiometer_Bourns_PTV09A-1_Single_Vertical, symbol Device:R_POT_TRIM
- removed SW101, SW102: FSM, Button_Switch_SMD:SW_Push_1P1T_NO_6x6mm_H9.5mm, symbol Switch:SW_MEC_5E
- added C103: 100nF, Capacitor_SMD:C_0805_2012Metric_Pad1.18x1.45mm_HandSolder, symbol Device:C
- added J101: Conn_01x11, Connector_PinHeader_2.54mm:PinHeader_1x11_P2.54mm_Vertical, symbol Connector_Generic:Conn_01x11
- added J104, J105: Conn_01x05, Connector_PinHeader_2.54mm:PinHeader_1x05_P2.54mm_Vertical, symbol Connector_Generic:Conn_01x05
- added R102, R103: 1K, Resistor_SMD:R_0805_2012Metric_Pad1.20x1.40mm_HandSolder, symbol Device:R
- C106: value 1uF -> 100nF
- J102: renamed from J101; footprint Connector_PinSocket_2.54mm:PinSocket_1x05_P2.54mm_Vertical -> Connector_PinHeader_2.54mm:PinHeader_1x05_P2.54mm_Vertical
- J103: renamed from J102; footprint Connector_PinSocket_2.54mm:PinSocket_1x05_P2.54mm_Vertical -> Connector_PinHeader_2.54mm:PinHeader_1x05_P2.54mm_Vertical; symbol Connector_Generic:Conn_01x03 -> Connector_Generic:Conn_01x05
- renumbered C103 to C102, C105 to C104, C104 to C105, R102 to R104, R103 to R105, R104 to R106, R105 to R107, R106 to R108, U107 to U201
Connections:
- net +3V3: now also J103.4 (Pin_4), R102.1, R103.1
- net +5V: now also J103.5 (Pin_5), C103.1
- net GND: now also C103.2, J101.11 (Pin_11), J105.3 (Pin_3), J105.5 (Pin_5)
- net LEDS: now also J105.4 (Pin_4)
- net RES0_A1: now also J105.1 (Pin_1)
- net RES0_W1: now also J105.2 (Pin_2)
- net RES_0: now also J101.5 (Pin_5)
- net RES_1: now also J101.6 (Pin_6)
- net RES_2: now also J101.7 (Pin_7)
- net RES_3: now also J101.8 (Pin_8)
- net SW_0: now also J101.9 (Pin_9), R103.2
- net SW_1: now also J101.10 (Pin_10), R102.2
- net at U102.33 (IO21): no longer J103.2 (Pin_2)
- net at U102.36 (IO22): no longer J103.3 (Pin_3)
- net at U102.8 (IO32): now also J103.2 (Pin_2)
- net DRY_WET: now reaches C110.2, R108.2
- net DRY_WET: now also J104.5 (Pin_5)
- new net V_OFFSET: J103.3 (Pin_3)
- new net input/IN_0_IN+: J101.1 (Pin_1)
- new net input/IN_1_IN+: J101.2 (Pin_2)
- new net input/IN_2_IN+: J101.3 (Pin_3)
- new net input/IN_3_IN+: J101.4 (Pin_4)
- new net output/OUT_0_OUT: J104.1 (Pin_1)
- new net output/OUT_1_OUT: J104.2 (Pin_2)
- new net output/OUT_2_OUT: J104.3 (Pin_3)
- new net output/OUT_3_OUT: J104.4 (Pin_4)
- no-connect marks 9 -> 13
Other:
- removed sheet switches
- sheet input ports: added IN_0_IN+, IN_1_IN+, IN_2_IN+, IN_3_IN+; removed none
- sheet output ports: added OUT_0_OUT, OUT_1_OUT, OUT_2_OUT, OUT_3_OUT; removed none
- note removed: "Four WS2B12B daisy chained"
- note removed: "LEDs"
- note removed: "Switches"
- note removed: "Two tactile switches and one rotary knob with switch"
- moved on the sheet: C108, C109, U101, U105, U106

Commit message: more pcb tracked
Parts:
- added J106: Conn_01x05, Connector_PinHeader_2.54mm:PinHeader_1x05_P2.54mm_Vertical, symbol Connector_Generic:Conn_01x05
- J101: value Conn_01x11 -> Conn_01x06; footprint Connector_PinHeader_2.54mm:PinHeader_1x11_P2.54mm_Vertical -> Connector_PinHeader_2.54mm:PinHeader_1x05_P2.54mm_Vertical; symbol Connector_Generic:Conn_01x11 -> Connector_Generic:Conn_01x05
Connections:
- net +3V3: now also J103.2 (Pin_2); no longer J103.4 (Pin_4)
- net +5V: now also J103.1 (Pin_1); no longer J103.5 (Pin_5)
- net GND: no longer J101.11 (Pin_11)
- net RES_1: now also J106.1 (Pin_1); no longer J101.6 (Pin_6)
- net RES_2: now also J106.2 (Pin_2); no longer J101.7 (Pin_7)
- net RES_3: now also J106.3 (Pin_3); no longer J101.8 (Pin_8)
- net RES_~RS: now also U102.11 (IO26)
- net RES_~SHDN: now also U102.10 (IO25)
- net SPI2_CLK: now also U104.3 (SCK); no longer U105.2 (SCK)
- net SPI2_CS_1: now also U104.2 (~{CS}); no longer U105.1 (~{CS})
- net SPI2_CS_2: now also U102.28 (IO17)
- net SPI2_MISO: now also U104.5 (~{LDAC}); no longer U105.13 (SO)
- net SPI2_MOSI: now also U104.4 (SDI); no longer U105.3 (SI)
- net SPI3_CLK: now also U105.2 (SCK); no longer U104.3 (SCK)
- net SPI3_CS_1: now also U105.1 (~{CS}); no longer U104.2 (~{CS})
- net SPI3_MISO: now also U105.13 (SO); no longer U104.5 (~{LDAC})
- net SPI3_MOSI: now also U105.3 (SI); no longer U104.4 (SDI)
- net SW_0: now also J106.4 (Pin_4); no longer J101.9 (Pin_9)
- net SW_1: now also J106.5 (Pin_5); no longer J101.10 (Pin_10)
- net at U102.33 (IO21): now also J103.5 (Pin_5)
- net at U102.8 (IO32): now also J103.4 (Pin_4); no longer J103.2 (Pin_2)
- no-connect marks 13 -> 11

Commit message: all hardware finished
Connections:
- net IO_21: now reaches J103.5 (Pin_5), U102.33 (IO21)
- net IO_32: now reaches J103.4 (Pin_4), U102.8 (IO32)
Changed lines of the file:
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@@
+    (effects (font (size 1.27 1.27)) (justify right bottom))
+  )
+  (label "IO_21" (at 152.4 220.98 180)
     (effects (font (size 1.27 1.27)) (justify right bottom))
   )
@@
     (effects (font (size 1.27 1.27)) (justify left bottom))
   )
+  (label "IO_32" (at 151.765 236.22 180)
+    (effects (font (size 1.27 1.27)) (justify right bottom))
+  )
   (label "PROG_TX" (at 48.26 259.08 180)
