File: hardware/curly-memory-kicad/curly-memory-kicad.kicad_sch (KiCad schematic)
At the start: 30 parts, among them J101 Conn_01x06, J102 Conn_01x05, J103 Conn_01x05, J104 Conn_01x05, J105 Conn_01x05, J106 Conn_01x05, U101 MCP3008-I/SL, U102 ESP32-WROOM-32, U103 MCP4822-E/SN, U104 MCP4822-E/SN, U105 MCP42010-E/SL, U106 MCP42010-E/SL, U201 MCP6004

Commit message: gerbers genearted and mf/mfpn added for main board for build
Parts:
- C101, C103, C104, C105, C106, C108, C109: MF (none) -> Samsung; MFPN (none) -> CL21B104KBCNNNC; Material (none) -> X7R; Voltage (none) -> 50V
- C102, C110: MF (none) -> Samsung; MFPN (none) -> CL21B105KBFNNNE; Material (none) -> X7R; Voltage (none) -> 50V
- J101, J102, J103, J104, J105, J106: now left out of the parts list
- R101, R102, R103, R104, R105, R106: MF (none) -> Multicomp; MFPN (none) -> MCWR08X1001FTL; Tolerance (none) -> 1%
- R107: MF (none) -> Multicomp; MFPN (none) -> MCWR08X1000FTL; Tolerance (none) -> 1%
- R108: MF (none) -> Multicomp; MFPN (none) -> MCWR08X1003FTL; Tolerance (none) -> 1%
- U105, U106: value MCP42010-E/SL -> MCP42010-I/SL
- U201: value MCP6004 -> MCP6004-I/SL
