File: hardware/curly-memory-kicad/output.kicad_sch (KiCad schematic)
At the start: 33 parts, among them J301 Conn_01x01_Male, J302 Conn_01x01_Male, J303 Conn_01x01_Male, J304 Conn_01x01_Male, J305 AudioJack2, J306 AudioJack2, J307 AudioJack2, J308 AudioJack2, U301 MCP6004

Commit message: all components placed on the main board
Parts:
- removed C303: 22pF, Capacitor_SMD:C_0805_2012Metric_Pad1.18x1.45mm_HandSolder, symbol Device:C
- removed C307, C309, C310: 1uF, Capacitor_SMD:C_0805_2012Metric_Pad1.18x1.45mm_HandSolder, symbol Device:C
- removed J301, J302, J303, J304: Conn_01x01_Male, Connector_PinSocket_2.54mm:PinSocket_1x01_P2.54mm_Vertical, symbol Connector:Conn_01x01_Male
- removed J305, J306, J307, J308: AudioJack2, AudioJacks:Jack_3.5mm_QingPu_WQP-PJ398SM_Vertical, symbol Connector:AudioJack2_Ground_SwitchT
- removed R303: 47k, Resistor_SMD:R_0805_2012Metric_Pad1.20x1.40mm_HandSolder, symbol Device:R
- removed R307, R311: 100K, Resistor_SMD:R_0805_2012Metric_Pad1.20x1.40mm_HandSolder, symbol Device:R
- renumbered C304 to C303, C305 to C304, C306 to C305, C308 to C306, C311 to C309, C312 to C310, R304 to R303, R305 to R304, R306 to R305, R308 to R306, R309 to R307, R310 to R308, R312 to R309
Connections:
- net GND: no longer U301.12 (+)
- net OUT_0 renamed OUT_0_OUT
- net OUT_1 renamed OUT_1_OUT
- net OUT_2 renamed OUT_2_OUT
- no-connect marks 0 -> 3

Commit message: gerbers genearted and mf/mfpn added for main board for build
Parts:
- C301, C302, C303: MF (none) -> Samsung; MFPN (none) -> CL21C220JBANNNC; Material (none) -> CG0 / NP0; Voltage (none) -> 50V
- C304, C305, C306: MF (none) -> Samsung; MFPN (none) -> CL21B105KBFNNNE; Material (none) -> X7R; Voltage (none) -> 50V
- C309, C310: MF (none) -> Samsung; MFPN (none) -> CL21B104KBCNNNC; Material (none) -> X7R; Voltage (none) -> 50V
- R301, R302, R303: value 47k -> 47K; MF (none) -> Multicomp; MFPN (none) -> MCWR08X4702FTL; Tolerance (none) -> 1%
- R304, R305, R306, R307, R308, R309: MF (none) -> Multicomp; MFPN (none) -> MCWR08X1003FTL; Tolerance (none) -> 1%
- U301: value MCP6004 -> MCP6004-I/SL
