File: hardware/curly-memory-interface-board/curly-memory-interface-board.kicad_sch (KiCad schematic)
At the start: 28 parts, among them J1 AudioJack2, J10 AudioJack2, J11 AudioJack2, J12 Conn_01x05, J13 Conn_01x05, J14 Conn_01x05, J15 Conn_01x05, J16 Conn_01x05, J17 Conn_01x02, J18 Conn_01x05, J2 AudioJack2, J3 AudioJack2, J4 Conn_01x05, J5 Conn_01x05, J6 Conn_01x05, J7 Conn_01x05, J8 AudioJack2, J9 AudioJack2, SW1 FSM, SW2 FSM, SW3 FSM, SW4 FSM

Commit message: all hardware finished
Connections:
- net IO17 is gone; now on net +5V: J14.1 (Pin_1), J16.1 (Pin_1)
- net IO21 is gone; now on net +3V3: J14.2 (Pin_2), J16.2 (Pin_2)
- net +3V3: no longer J14.4 (Pin_4), J16.4 (Pin_4)
- net +5V: no longer J14.5 (Pin_5), J16.5 (Pin_5)
- net IO22 renamed V_OFFSET
- new net IO_21: J14.5 (Pin_5), J16.5 (Pin_5)
- new net IO_32: J14.4 (Pin_4), J16.4 (Pin_4)
Changed lines of the file:
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@@
   (junction (at 168.91 63.5) (diameter 0) (color 0 0 0 0)
   )
-  (junction (at 212.725 222.25) (diameter 0) (color 0 0 0 0)
+  (junction (at 209.55 217.17) (diameter 0) (color 0 0 0 0)
   )
   (junction (at 152.4 224.79) (diameter 0) (color 0 0 0 0)
@@
   (junction (at 46.99 43.815) (diameter 0) (color 0 0 0 0)
   )
+  (junction (at 205.74 219.71) (diameter 0) (color 0 0 0 0)
+  )
   (junction (at 168.91 44.45) (diameter 0) (color 0 0 0 0)
   )
@@
   (junction (at 168.91 82.55) (diameter 0) (color 0 0 0 0)
   )
-  (junction (at 206.375 224.79) (diameter 0) (color 0 0 0 0)
+  (junction (at 214.63 214.63) (diameter 0) (color 0 0 0 0)
   )
   (no_connect (at 326.39 64.135))
@@
     (stroke (width 0) (type default) (color 0 0 0 0))
   )
-  (wire (pts (xy 206.375 224.79) (xy 206.375 229.87))
-    (stroke (width 0) (type default) (color 0 0 0 0))
-  )
-  (wire (pts (xy 201.295 224.79) (xy 206.375 224.79))
+  (wire (pts (xy 214.63 214.63) (xy 214.63 209.55))
+    (stroke (width 0) (type default) (color 0 0 0 0))
+  )
+  (wire (pts (xy 219.71 214.63) (xy 214.63 214.63))
     (stroke (width 0) (type default) (color 0 0 0 0))
   )
@@
     (stroke (width 0) (type default) (color 0 0 0 0))
   )
-  (wire (pts (xy 212.725 222.25) (xy 201.295 222.25))
-    (stroke (width 0) (type default) (color 0 0 0 0))
-  )
-  (wire (pts (xy 201.295 214.63) (xy 219.71 214.63))
+  (wire (pts (xy 209.55 217.17) (xy 219.71 217.17))
     (stroke (width 0) (type default) (color 0 0 0 0))
   )
@@
     (stroke (width 0) (type default) (color 0 0 0 0))
   )
-  (wire (pts (xy 201.295 219.71) (xy 219.71 219.71))
+  (wire (pts (xy 201.295 219.71) (xy 205.74 219.71))
     (stroke (width 0) (type default) (color 0 0 0 0))
   )
@@
     (stroke (width 0) (type default) (color 0 0 0 0))
   )
+  (wire (pts (xy 205.74 219.71) (xy 219.71 219.71))
+    (stroke (width 0) (type default) (color 0 0 0 0))
+  )
   (wire (pts (xy 55.245 77.47) (xy 55.245 46.355))
     (stroke (width 0) (type default) (color 0 0 0 0))
@@
     (stroke (width 0) (type default) (color 0 0 0 0))
   )
-  (wire (pts (xy 206.375 224.79) (xy 219.71 224.79))
+  (wire (pts (xy 214.63 214.63) (xy 201.295 214.63))
     (stroke (width 0) (type default) (color 0 0 0 0))
   )
@@
     (stroke (width 0) (type default) (color 0 0 0 0))
   )
-  (wire (pts (xy 212.725 229.87) (xy 212.725 222.25))
+  (wire (pts (xy 209.55 209.55) (xy 209.55 217.17))
+    (stroke (width 0) (type default) (color 0 0 0 0))
+  )
+  (wire (pts (xy 201.295 222.25) (xy 219.71 222.25))
     (stroke (width 0) (type default) (color 0 0 0 0))
   )
@@
     (stroke (width 0) (type default) (color 0 0 0 0))
   )
-  (wire (pts (xy 212.725 222.25) (xy 219.71 222.25))
+  (wire (pts (xy 205.74 211.455) (xy 205.74 219.71))
+    (stroke (width 0) (type default) (color 0 0 0 0))
+  )
+  (wire (pts (xy 209.55 217.17) (xy 201.295 217.17))
     (stroke (width 0) (type default) (color 0 0 0 0))
   )
@@
     (stroke (width 0) (type default) (color 0 0 0 0))
   )
-  (wire (pts (xy 201.295 217.17) (xy 219.71 217.17))
-    (stroke (width 0) (type default) (color 0 0 0 0))
-  )
   (wire (pts (xy 49.53 82.55) (xy 49.53 84.455))
     (stroke (width 0) (type default) (color 0 0 0 0))
@@
   )
   (wire (pts (xy 144.78 217.17) (xy 167.005 217.17))
+    (stroke (width 0) (type default) (color 0 0 0 0))
+  )
+  (wire (pts (xy 201.295 224.79) (xy 219.71 224.79))
     (stroke (width 0) (type default) (color 0 0 0 0))
   )
@@
     (effects (font (size 1.27 1.27) italic) (justify left bottom))
   )
-  (label "IO21" (at 205.74 217.17 0)
-    (effects (font (size 1.27 1.27)) (justify left bottom))
-  )
   (label "IN_3" (at 66.675 85.09 0)
     (effects (font (size 1.27 1.27)) (justify left bottom))
@@
     (effects (font (size 1.27 1.27)) (justify left bottom))
   )
+  (label "IO_32" (at 208.915 222.25 0)
+    (effects (font (size 1.27 1.27)) (justify left bottom))
+  )
   (label "SW_1" (at 66.675 101.6 0)
     (effects (font (size 1.27 1.27)) (justify left bottom))
@@
     (effects (font (size 1.27 1.27)) (justify left bottom))
   )
-  (label "IO22" (at 205.74 219.71 0)
-    (effects (font (size 1.27 1.27)) (justify left bottom))
-  )
   (label "IN_1" (at 66.675 80.01 0)
     (effects (font (size 1.27 1.27)) (justify left bottom))
@@
     (effects (font (size 1.27 1.27)) (justify left bottom))
   )
-  (label "IO17" (at 205.74 214.63 0)
-    (effects (font (size 1.27 1.27)) (justify left bottom))
-  )
   (label "SW_1" (at 296.545 168.91 0)
     (effects (font (size 1.27 1.27)) (justify left bottom))
@@
   )
   (label "RST" (at 327.66 154.94 0)
+    (effects (font (size 1.27 1.27)) (justify left bottom))
+  )
+  (label "IO_21" (at 208.915 224.79 0)
     (effects (font (size 1.27 1.27)) (justify left bottom))
   )
@@
   )
   (label "SW_0" (at 296.545 154.94 0)
+    (effects (font (size 1.27 1.27)) (justify left bottom))
+  )
+  (label "V_OFFSET" (at 205.74 211.455 90)
     (effects (font (size 1.27 1.27)) (justify left bottom))
   )
@@
     (pin "5")
   )
-  (symbol (lib_name "+5V_1") (lib_id "power:+5V") (at 206.375 229.87 180) (unit 1)
-    (in_bom yes) (on_board yes) (fields_autoplaced)
-    (property "Reference" "#PWR019" (id 0) (at 206.375 226.06 0)
-      (effects (font (size 1.27 1.27)) hide)
-    )
-    (property "Value" "+5V" (id 1) (at 206.375 234.4325 0))
-    (property "Footprint" "" (id 2) (at 206.375 229.87 0)
-      (effects (font (size 1.27 1.27)) hide)
-    )
-    (property "Datasheet" "" (id 3) (at 206.375 229.87 0)
+  (symbol (lib_name "+5V_1") (lib_id "power:+5V") (at 214.63 209.55 0) (unit 1)
+    (in_bom yes) (on_board yes) (fields_autoplaced)
+    (property "Reference" "#PWR019" (id 0) (at 214.63 213.36 0)
+      (effects (font (size 1.27 1.27)) hide)
+    )
+    (property "Value" "+5V" (id 1) (at 214.63 204.9875 0))
+    (property "Footprint" "" (id 2) (at 214.63 209.55 0)
+      (effects (font (size 1.27 1.27)) hide)
+    )
+    (property "Datasheet" "" (id 3) (at 214.63 209.55 0)
       (effects (font (size 1.27 1.27)) hide)
     )
@@
     (pin "TN")
   )
-  (symbol (lib_id "power:+3V3") (at 212.725 229.87 180) (unit 1)
-    (in_bom yes) (on_board yes) (fields_autoplaced)
-    (property "Reference" "#PWR021" (id 0) (at 212.725 226.06 0)
-      (effects (font (size 1.27 1.27)) hide)
-    )
-    (property "Value" "+3V3" (id 1) (at 212.725 234.4325 0))
-    (property "Footprint" "" (id 2) (at 212.725 229.87 0)
-      (effects (font (size 1.27 1.27)) hide)
-    )
-    (property "Datasheet" "" (id 3) (at 212.725 229.87 0)
-      (effects (font (size 1.27 1.27)) hide)
-    )
+  (symbol (lib_id "power:+3V3") (at 209.55 209.55 0) (unit 1)
+    (in_bom yes) (on_board yes) (fields_autoplaced)
+    (property "Reference" "#PWR021" (id 0) (at 209.55 213.36 0)
+      (effects (font (size 1.27 1.27)) hide)
+    )
+    (property "Value" "+3V3" (id 1) (at 209.55 204.9875 0))
+    (property "Footprint" "" (id 2) (at 209.55 209.55 0)
+      (effects (font (size 1.27 1.27)) hide)
+    )
+    (property "Datasheet" "" (id 3) (at 209.55 209.55 0)
+      (effects (font (size 1.27 1.27)) hide)
+    )
