File: hardware/curly-memory-face-plate/curly-memory-face-plate.kicad_pcb (KiCad board)
At the start: 2 copper layers, 30 x 129 mm, 23 parts, among them J1 Thonkiconn_PJ398SM_panel, J2 Thonkiconn_PJ398SM_panel, J3 Thonkiconn_PJ398SM_panel, J4 Thonkiconn_PJ398SM_panel, J5 Thonkiconn_PJ398SM_panel, J6 Thonkiconn_PJ398SM_panel, J7 Thonkiconn_PJ398SM_panel, P1 2.54_pinheader_panel_01x05, P2 2.54_pinheader_panel_01x05, P3 2.54_pinheader_panel_01x05, P4 2.54_pinheader_panel_01x05, SW1 FSM14J_panel, SW2 FSM14J_panel, SW3 FSM14J_panel, SW4 FSM14J_panel

Commit message: all hardware finished
Parts:
- moved J1 0.50 mm to (22.5, 85.0)
Other:
- board text added: "3V3"
- board text added: "5V"
- board text added: "BOOT"
- board text added: "DRY WET"
- board text added: "GND"
- board text added: "IN 0"
- board text added: "IN 1"
- board text added: "IN 2"
- board text added: "IN 3"
- board text added: "IO22"
- board text added: "IO32"
- board text added: "LEDS"
- board text added: "OFFSET"
- board text added: "OUT 0"
- board text added: "OUT 1"
- board text added: "OUT 2"
- board text added: "OUT 3"
- board text added: "RES A"
- board text added: "RES B"
- board text added: "RES W"
- board text added: "RST"
- board text added: "RV1"
- board text added: "RV2"
- board text added: "RV3"
- board text added: "RV4"
- board text added: "RX"
- board text added: "SW0"
- board text added: "SW1"
- board text added: "TX"
- board text added: "V"
- board text added: "curly memory"
- board text added: "r f e"
- board text added: "ric from ealing"
Changed lines of the file:
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@@
   (setup
     (pad_to_mask_clearance 0)
+    (grid_origin 5.715 58.42)
     (pcbplotparams
       (layerselection 0x00010fc_ffffffff)
@@
   )
   (footprint "mylibs6:Thonkiconn_PJ398SM_panel" (layer "F.Cu")
-    (at 22.5 85.5)
+    (at 22.5 85)
     (property "Sheetfile" "curly-memory-face-plate.kicad_sch")
     (property "Sheetname" "")
@@
     (pad "" np_thru_hole circle (at 0 0) (size 6.1 6.1) (drill 6.1) (layers *.Cu *.Mask))
   )
+  (gr_circle (center 22.5 62.5) (end 25 62.5) (layer "B.Mask") (width 0.15) (fill solid))
+  (gr_circle (center 7.5 62.5) (end 10 62.5) (layer "B.Mask") (width 0.15) (fill solid))
   (gr_circle (center 22.5 62.5) (end 25 62.5) (layer "F.Mask") (width 0.15) (fill solid))
   (gr_circle (center 7.5 62.5) (end 10 62.5) (layer "F.Mask") (width 0.15) (fill solid))
@@
   (gr_line (start 30 -14.5) (end 30 114.5) (layer "Edge.Cuts") (width 0.1))
   (gr_line (start 0 114.5) (end 30 114.5) (layer "Edge.Cuts") (width 0.1))
+  (gr_text "RES A" (at 2.54 76.835 90) (layer "F.SilkS")
+    (effects (font (size 0.75 0.75) (thickness 0.15)) (justify right))
+  )
+  (gr_text "OUT 2" (at 25.16 76.835 90) (layer "F.SilkS")
+    (effects (font (size 0.75 0.75) (thickness 0.15)) (justify right))
+  )
+  (gr_text "OUT 2" (at 7.5 99.85) (layer "F.SilkS")
+    (effects (font (size 1 1) (thickness 0.15)))
+  )
+  (gr_text "RST" (at 5.08 70.485 90) (layer "F.SilkS")
+    (effects (font (size 0.75 0.75) (thickness 0.15)) (justify right))
+  )
+  (gr_text "IN 0" (at 7.5 40.55) (layer "F.SilkS")
+    (effects (font (size 1 1) (thickness 0.15)))
+  )
+  (gr_text "IO22" (at 27.7 70.485 90) (layer "F.SilkS")
+    (effects (font (size 0.75 0.75) (thickness 0.15)) (justify right))
+  )
+  (gr_text "RV2" (at 22.86 11.65) (layer "F.SilkS")
+    (effects (font (size 1 1) (thickness 0.15)))
+  )
+  (gr_text "RV3" (at 7.62 26.35) (layer "F.SilkS")
+    (effects (font (size 1 1) (thickness 0.15)))
+  )
+  (gr_text "OUT 0" (at 7.5 89.95) (layer "F.SilkS")
+    (effects (font (size 1 1) (thickness 0.15)))
+  )
+  (gr_text "BOOT" (at 4.5 58.674) (layer "F.SilkS")
+    (effects (font (size 0.75 0.75) (thickness 0.15)))
+  )
+  (gr_text "GND" (at 12.7 70.485 90) (layer "F.SilkS")
+    (effects (font (size 0.75 0.75) (thickness 0.15)) (justify right))
+  )
+  (gr_text "r\nf\ne" (at 15 106.045) (layer "F.SilkS")
+    (effects (font (size 1 1) (thickness 0.15)))
+  )
+  (gr_text "DRY WET" (at 22.5 99.85) (layer "F.SilkS")
+    (effects (font (size 1 1) (thickness 0.15)))
+  )
+  (gr_text "IN 3" (at 17.54 76.835 90) (layer "F.SilkS")
+    (effects (font (size 0.75 0.75) (thickness 0.15)) (justify right))
+  )
+  (gr_text "3V3" (at 20.08 70.485 90) (layer "F.SilkS")
+    (effects (font (size 0.75 0.75) (thickness 0.15)) (justify right))
+  )
+  (gr_text "IN 2" (at 22.62 76.835 90) (layer "F.SilkS")
+    (effects (font (size 0.75 0.75) (thickness 0.15)) (justify right))
+  )
+  (gr_text "RST" (at 11.5 58.674) (layer "F.SilkS")
+    (effects (font (size 0.75 0.75) (thickness 0.15)))
+  )
+  (gr_text "GND" (at 12.7 76.835 90) (layer "F.SilkS")
+    (effects (font (size 0.75 0.75) (thickness 0.15)) (justify right))
+  )
+  (gr_text "curly memory" (at 15 -8) (layer "F.SilkS")
+    (effects (font (size 1 1) (thickness 0.15)))
+  )
+  (gr_text "TX" (at 7.62 70.485 90) (layer "F.SilkS")
+    (effects (font (size 0.75 0.75) (thickness 0.15)) (justify right))
+  )
+  (gr_text "5V" (at 17.54 70.485 90) (layer "F.SilkS")
+    (effects (font (size 0.75 0.75) (thickness 0.15)) (justify right))
+  )
+  (gr_text "SW1" (at 25.5 58.674) (layer "F.SilkS")
+    (effects (font (size 0.75 0.75) (thickness 0.15)))
+  )
+  (gr_text "LEDS" (at 10.16 76.835 90) (layer "F.SilkS")
+    (effects (font (size 0.75 0.75) (thickness 0.15)) (justify right))
+  )
+  (gr_text "RV4" (at 22.86 26.35) (layer "F.SilkS")
+    (effects (font (size 1 1) (thickness 0.15)))
+  )
+  (gr_text "IN 1" (at 7.5 50.65) (layer "F.SilkS")
+    (effects (font (size 1 1) (thickness 0.15)))
+  )
+  (gr_text "GND" (at 27.7 76.835 90) (layer "F.SilkS")
+    (effects (font (size 0.75 0.75) (thickness 0.15)) (justify right))
+  )
+  (gr_text "BOOT" (at 2.54 70.485 90) (layer "F.SilkS")
+    (effects (font (size 0.75 0.75) (thickness 0.15)) (justify right))
+  )
+  (gr_text "RES B" (at 7.62 76.835 90) (layer "F.SilkS")
+    (effects (font (size 0.75 0.75) (thickness 0.15)) (justify right))
+  )
+  (gr_text "OFFSET" (at 22.86 71.755 90) (layer "F.SilkS")
+    (effects (font (size 0.5 0.5) (thickness 0.125)))
+  )
+  (gr_text "V" (at 22.62 73.025 90) (layer "F.SilkS")
+    (effects (font (size 0.75 0.75) (thickness 0.15)) (justify right))
+  )
+  (gr_text "RX" (at 10.16 70.485 90) (layer "F.SilkS")
+    (effects (font (size 0.75 0.75) (thickness 0.15)) (justify right))
+  )
+  (gr_text "OUT 1" (at 22.5 89.95) (layer "F.SilkS")
+    (effects (font (size 1 1) (thickness 0.15)))
+  )
+  (gr_text "RV1" (at 7.62 11.65) (layer "F.SilkS")
+    (effects (font (size 1 1) (thickness 0.15)))
+  )
+  (gr_text "ric from ealing" (at 15 -4) (layer "F.SilkS")
+    (effects (font (size 1 1) (thickness 0.15)))
+  )
+  (gr_text "RES W" (at 5.08 76.835 90) (layer "F.SilkS")
+    (effects (font (size 0.75 0.75) (thickness 0.15)) (justify right))
+  )
+  (gr_text "IN 2" (at 22.5 50.65) (layer "F.SilkS")
+    (effects (font (size 1 1) (thickness 0.15)))
+  )
+  (gr_text "SW0" (at 18.5 58.674) (layer "F.SilkS")
+    (effects (font (size 0.75 0.75) (thickness 0.15)))
+  )
+  (gr_text "IO32" (at 25.16 70.485 90) (layer "F.SilkS")
+    (effects (font (size 0.75 0.75) (thickness 0.15)) (justify right))
+  )
+  (gr_text "OUT 3" (at 20.08 76.835 90) (layer "F.SilkS")
+    (effects (font (size 0.75 0.75) (thickness 0.15)) (justify right))
+  )
 )
